File: Avada_hw/avada.sch (KiCad schematic (older format))
At the start: 40 parts

Commit message: + Avada4 sent to production
Parts:
- removed Logo?: Logo, Pictures:Ostranna_12d7_10d1, symbol Logo
- removed TP?: TESTPOINT, PCB:TESTPOINT_1MM, symbol TESTPOINT
- added D4: LED, LEDs:LED_RAD, symbol LED
- added D5: LED, LEDs:LED_XPE, symbol LED
- D3: renamed from D?; footprint LEDs:LED_Through-Hole-5mm-HOR -> LEDs:LED_Diamond_Dragon; PN TSAL6200 -> (none); URL https://www.terraelectronica.ru/catalog_info.php?CODE=31376 -> (none)
- SW2: renamed from SW?; footprint Switches:DIP_SMD_1D27X6 -> BtnsSwitches:DIP_SMD_1D27X6
- gave numbers to parts that had none: 36
Connections:
- wire segments 131 -> 134
- no-connect marks 25 -> 26
Other:
- note added: "One or another"

Commit message: Switch to Atollic
Parts:
- B1: symbol BAT -> Power_kl:BAT
- BZ1: symbol BUZZER -> Tittar_kl:BUZZER
- C1, C10, C11, C2, C3, C4, C5, C6, C7, C8, C9: symbol C -> Tittar_kl:C
- C12, C13: symbol CP -> Tittar_kl:CP
- D1, D3, D4, D5: symbol LED -> Tittar_kl:LED
- D2: symbol D_Shottky -> Tittar_kl:D_Shottky
- DA1: symbol MCP73832 -> Power_kl:MCP73832
- DA2: symbol NCP583SQ -> Power_kl:NCP583SQ
- DD1: symbol STM32L151CxTx -> st_kl:STM32L151CxTx
- F1: symbol Fuse0R -> Tittar_kl:Fuse0R
- Q1, Q2: symbol P_3PIN -> Transistors_kl:P_3PIN
- Q3, Q4, Q5: symbol NPN -> Transistors_kl:NPN
- R1, R2, R3, R4, R5, R6: symbol R -> Tittar_kl:R
- SW1: symbol BUTTON -> Switches:BUTTON
- SW2: symbol DIPx6 -> Switches:DIPx6
- SW3: symbol SWITCH -> Switches:SWITCH
- XL1: symbol CONN_6 -> Connectors_kl:CONN_6
- XL2: symbol USB_MINI_B -> Connectors_kl:USB_MINI_B
Connections:
- wire segments 134 -> 176
