File: Avada_hw/Avada.kicad_sch (KiCad schematic)
At the start: 52 parts, among them Q1 IRLML6401, Q2 DMG2302, Q4 DMG2302, Q5 IRLML6401, SW1 IT1198

Commit message: Sch seems done
Parts:
- removed C14: 3F, Capacitors:CAP_08xxR_HOR, symbol Tittar_kl:CP
- removed C15: 2u2, Capacitors:CAP_0603_Silks, symbol Tittar_kl:C
- removed D4: LEDwPAD, LEDs:LED_XPE, symbol Tittar_kl:LEDwPAD
- removed Q4: DMG2302, SOT:SOT23-3A, symbol Transistors_kl:N_3PIN
- removed Q5: IRLML6401, SOT:SOT23-3, symbol Transistors_kl:P_3PIN
- removed R1: 5k1, Resistors:RES_0603, symbol Tittar_kl:R
- removed R14, R16, R17, R18: 56k, Resistors:RES_0603, symbol Tittar_kl:R
- removed R15: 0R1, Resistors:RES_1206, symbol Tittar_kl:R
- removed R19: 2R0, Resistors:RES_0603, symbol Tittar_kl:R
- removed XL3: USB_C, Connectors:USB_C_MOLEX_1054500101, symbol Connectors_kl:USB_C
- added C12: 2u2, Capacitors:CAP_0603_Silks, symbol Tittar_kl:C
- added C2, C3: 1u, Capacitors:CAP_0603_Silks, symbol Tittar_kl:C
- added D1, D10, D11, D12, D13, D14, D15, D16, D17, D18, D19, D2, D20, D3, D4, D5, D6, D7, D8, D9: 2835, LEDs:LED_PLCC2835, symbol Tittar_kl:LED
- added DA1: MCP1700-3002, SOT:SOT23-3A, symbol Power_kl:MCP1700
- added Q1: IRLML6401, SOT:SOT23-3, symbol Transistors_kl:P_3PIN
- added R11, R8: 56k, Resistors:RES_0603, symbol Tittar_kl:R
- added R4, R7: 5k1, Resistors:RES_0603, symbol Tittar_kl:R
- added R6: 2R0, Resistors:RES_0603, symbol Tittar_kl:R
- added XL2: 10PF-074, Connectors:USBC_10PF-074, symbol Connectors_kl:USBC-16P
- R2: value 5k1 -> 56k
- renumbered C13 to C1, C7 to C10, C8 to C11, C11 to C13, C12 to C14, C9 to C15, C10 to C16, C1 to C4, C2 to C5, C3 to C6, C4 to C7, C5 to C8, C6 to C9, D1 to D21, D2 to D22, DA1 to DA3, HOLE3 to HOLE1, HOLE4 to HOLE3, HOLE1 to HOLE4, Q1 to Q3, R12 to R1, R4 to R10, R7 to R12, R5 to R13, R8 to R5, R6 to R9, XL4 to XL3, XL2 to XL4
Connections:
- net +5V_USB: now also R6.1, XL2.A4B9 (VBUS), XL2.B4A9 (VBUS)
- net +BATT: now also C2.1, DA1.3 (IN), R8.1; no longer R1.1
- net GND: now also C1.2, C12.2, C2.2, C3.2, D1.C, D10.C, D11.C, D12.C, D13.C, D14.C, D15.C, D16.C, D17.C, D18.C, D19.C, D2.C, D20.C, D3.C, D4.C, D5.C, D6.C, D7.C, D8.C, D9.C, DA1.1 (GND), R4.1, R7.2, XL2.A1B12 (GND), XL2.B1A12 (GND); no longer R2.1
- net LED_CTRL: now also R2.2, Q1.1 (G)
- net USB_D+: now also XL2.A6 (DP1), XL2.B6 (DP2)
- net USB_D-: now also XL2.A7 (DN1), XL2.B7 (DN2)
- net at C1.1, R1.2: now also R2.1, Q1.2 (S)
- net ADC_BAT_EN: now reaches DD1.28 (PB2)
- net ADC_BAT_EN: now also R11.2
- net LED_CURR: no longer names the net of DD1.17 (ADC3/T15C2/T2C4/RX2/PA3)
- net LED_V: no longer names the net of DD1.16 (ADC2/T15C1/T2C3/TX2/PA2)
- net MeasEn renamed ADC_BAT
- net ADC_BAT: now also R11.1, R8.2
- new net: D1.A, D10.A, D11.A, D12.A, D13.A, D14.A, D15.A, D16.A, D17.A, D18.A, D19.A, D2.A, D20.A, D3.A, D4.A, D5.A, D6.A, D7.A, D8.A, D9.A, Q1.3 (D)
- new net: C3.1, DA1.2 (OUT), R1.1
- new net: C12.1, R6.2
- new net USB_CC1_IN: R4.2, XL2.A5 (CC1)
- new net USB_CC2_IN: R7.1, XL2.B5 (CC2)
- no-connect marks 54 -> 46
Other:
- note added: "3V 20R => 150mA max"
- note added: "3V power"
- note added: "5v tolerant"
- note added: "Battery Measurement"
- note added: "Bright Green"
- note added: "Power"
- note added: "Sound"
- note added: "T14C1 or DAC1"
- note added: "USB-C connector"
- note added: "Use 3V or 3V3 MCP1700"
- note removed: "3V 20R => 150mA"
- moved on the sheet: BZ1, C1, C13, C14, C15, C16, D22, DA2, DA3, HOLE1, HOLE2, HOLE3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

Commit message: PCB Layout Started
Parts:
- removed HOLE1, HOLE2, HOLE3, HOLE4: HOLE_METALLED, PCB:Hole2d2_out3d5mm, symbol pcb_details:HOLE_METALLED
- removed Q1: IRLML6401, SOT:SOT23-3, symbol Transistors_kl:P_3PIN
- added D21: 2835, LEDs:LED_PLCC2835, symbol Tittar_kl:LED
- added Q1: IRLML0030, SOT:SOT23-3, symbol Transistors_kl:N_3PIN
- Q2: footprint SOT:SOT23-3A -> SOT:SOT23-3
- renumbered C2 to C1, C3 to C2, C1 to C3, D21 to D22, D22 to D23
Connections:
- net GND: now also R2.2, Q1.2 (S); no longer D1.C, D10.C, D11.C, D12.C, D13.C, D14.C, D15.C, D16.C, D17.C, D18.C, D19.C, D2.C, D20.C, D3.C, D4.C, D5.C, D6.C, D7.C, D8.C, D9.C
- net LED_CTRL: now also R2.1, Q1.1 (G); no longer R2.2
- net at D1.A, D10.A, D11.A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: now also C3.1, R1.2, D21.A
- new net: D1.C, D10.C, D11.C, D12.C, D13.C, D14.C, D15.C, D16.C, D17.C, D18.C, D19.C, D2.C, D20.C, D21.C, D3.C, D4.C, D5.C, D6.C, D7.C, D8.C, D9.C, Q1.3 (D)
Other:
- moved on the sheet: C1, C2, C3, D1, D10, D11, D12, D13, D14, D15, D16, D17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

Commit message: + PCB sent to factory
Parts:
- removed C3: 3F, Capacitors:CAP_08xxR_HOR, symbol Tittar_kl:CP
- removed XL4: CONN_2, Connectors:SLD_2_2D5, symbol Connectors_kl:CONN_2
- added XL4: CONN_1, Connectors:PLS-1Oval, symbol Connectors_kl:CONN_1
- added XL5, XL6: CONN_1, Connectors:PLS-1Square, symbol Connectors_kl:CONN_1
- added XL7: CONN_1, Connectors:PLS-1Rnd, symbol Connectors_kl:CONN_1
Connections:
- net +BATT: now also SA1.1, XL4.1 (P1); no longer SA1.3
- net GND: now also XL5.1 (P1), XL6.1 (P1)
- net +PwrLED: now reaches D1.A, D10.A, D11.A, D12.A, D13.A, D14.A, D15.A, D16.A, D17.A, D18.A, D19.A, D2.A, D20.A, D21.A, D3.A, D4.A, D5.A, D6.A, D7.A, D8.A, D9.A, R1.2
- net +PwrLED: now also XL7.1 (P1)
- net -PwrLED: now reaches D1.C, D10.C, D11.C, D12.C, D13.C, D14.C, D15.C, D16.C, D17.C, D18.C, D19.C, D2.C, D20.C, D21.C, D3.C, D4.C, D5.C, D6.C, D7.C, D8.C, D9.C, Q1.3 (D)
- net +3vLED: now reaches C2.1, DA1.2 (OUT), R1.1
Other:
- note added: "Ionistor 3V 3F"
- moved on the sheet: C13, C14
