File: Avada_hw/avada.kicad_pcb (KiCad board)
At the start: 2 copper layers, 30.2 x 53.5 mm, 40 parts, among them Q1 IRLML6401, Q2 IRLML6401, Q3 NSS20101, Q4 NSS20101, Q5 NSS20101, SW1 IT1198, SW2 DIPx6, SW3 SS-1P2T

Commit message: Some renamings
Parts:
- removed B1: LP603030, Installation:EEMB603030
- removed D3: LED, LEDs:LED_Diamond_Dragon
- removed D5: LED, LEDs:LED_XPE
- removed F1: Fuse0R, Resistors:RES_0603_FUSE
- removed Q3: NSS20101, SOT:SC89-3
- removed SW2: DIPx6, BtnsSwitches:DIP_SMD_1D27X6
- removed SW3: SS-1P2T, BtnsSwitches:SW_SS-1P2T_R
- added C14: 3F, Capacitors:CAP_08xxR_HOR, F.Cu at (160.6, 86.2)
- added C15: 2u2, Capacitors:CAP_0603_Silks, F.Cu at (152.6, 112.0)
- added HOLE1: HOLE_METALLED, PCB:Hole2d2_out3d5mm, F.Cu at (153.3, 116.7)
- added HOLE2: HOLE_METALLED, PCB:Hole2d2_out3d5mm, F.Cu at (129.3, 58.7)
- added HOLE3: HOLE_METALLED, PCB:Hole2d2_out3d5mm, F.Cu at (129.3, 116.7)
- added HOLE4: HOLE_METALLED, PCB:Hole2d2_out3d5mm, F.Cu at (162.3, 58.7)
- added L1: BLM15AG102, Inductors:IND_0402, F.Cu at (159.5, 74.1)
- added R12: 20R, Resistors:RES_0603, F.Cu at (143.5, 71.1)
- added R14: 56k, Resistors:RES_0603, F.Cu at (149.1, 62.5)
- added R15: 0R1, Resistors:RES_1206, F.Cu at (147.0, 59.8)
- added R16: 56k, Resistors:RES_0603, F.Cu at (142.0, 68.4)
- added R17: 56k, Resistors:RES_0603, F.Cu at (139.4, 65.5)
- added R18: 56k, Resistors:RES_0603, F.Cu at (139.4, 68.5)
- added R19: 2R0, Resistors:RES_0603, F.Cu at (152.6, 110.5)
- added R7: 3k, Resistors:RES_0603, F.Cu at (139.9, 116.6)
- added R8: 56k, Resistors:RES_0603, F.Cu at (150.9, 66.3)
- added SA1: SS-12F23, BtnsSwitches:SW_SS-12F23, F.Cu at (137.1, 68.2)
- added XL3: USB_C, Connectors:USB_C_MOLEX_1054500101, F.Cu at (145.8, 119.3)
- added XL4: CONN_1, Connectors:PLS-1Square, F.Cu at (128.3, 110.1)
- C1: value 10n -> 10u; footprint Capacitors:CAP_0603 -> Capacitors:CAP_0603_Silks; moved to F.Cu
- C10: value 10n -> 1u; footprint Capacitors:CAP_0603 -> Capacitors:CAP_0603_Silks; moved to F.Cu
- C11: value 1u -> 10u; footprint Capacitors:CAP_0603 -> Capacitors:CAP_0603_Silks; moved to F.Cu
- C12: value 220u -> 10u; footprint Capacitors:CAP_05xxR_horiz_HOLE -> Capacitors:CAP_0603_Silks; moved to F.Cu
- C13: value 220u -> 3F; footprint Capacitors:CAP_05xxR_horiz_HOLE -> Capacitors:CAP_08xxR_HOR; moved to F.Cu
- C2, C4, C6: value 10u -> 0.1u; footprint Capacitors:CAP_0603 -> Capacitors:CAP_0603_Silks; moved to F.Cu
- C3, C5: value 1u -> 0.1u; footprint Capacitors:CAP_0603 -> Capacitors:CAP_0603_Silks; moved to F.Cu
- C7: value 0.1u -> 10n; footprint Capacitors:CAP_0603 -> Capacitors:CAP_0603_Silks; moved to F.Cu
- C8, C9: value 0.1u -> 1u; footprint Capacitors:CAP_0603 -> Capacitors:CAP_0603_Silks; moved to F.Cu
- D1: value LED -> L-C191LBCT; moved to F.Cu
- D4: value LED -> LEDwPAD; footprint LEDs:LED_RAD -> LEDs:LED_XPE
- DA1: value MCP73832 -> MCP1700; footprint SOT:SOT23-5 -> SOT:SOT23-3A; moved to F.Cu
- DA2: value NCP583SQ -> TP4056; footprint SOT:SC82AB -> SO_DIL_TSSOP:SO8_150MIL; moved to F.Cu
- DD1: value STM32L151CxTx -> STM32F072RxTx; footprint LQFP_TQFP:LQFP48 -> LQFP_TQFP:LQFP64; moved to F.Cu
- Q2: value IRLML6401 -> DMG2302; footprint SOT:SOT23-3 -> SOT:SOT23-3A
- Q4: value NSS20101 -> DMG2302; footprint SOT:SC89-3 -> SOT:SOT23-3A
- Q5: value NSS20101 -> IRLML6401; footprint SOT:SC89-3 -> SOT:SOT23-3; moved to F.Cu
- R1: value 1k -> 5k1; moved to F.Cu
- R2: value 3k -> 5k1; moved to F.Cu
- R3: value 10k -> 1k; moved to F.Cu
- R4: moved to F.Cu
- R5: value 1k -> 10k; moved to F.Cu
- R6: value 1k -> 0R2; footprint Resistors:RES_0603 -> Resistors:RES_1206; moved to F.Cu
- XL2: value USB_Micro_B -> CONN_2; footprint Connectors:USBmicro_MOLEX_WM17142 -> Connectors:SLD_2_2D5; moved to F.Cu
- moved XL1 62.4 mm to (163.5, 71.3)
- moved C8 57.4 mm to (161.4, 75.0), turned to 90 degrees
- moved DA1 55.7 mm to (139.9, 59.6)
- moved C1 54.5 mm to (153.7, 69.0), turned to 180 degrees
- moved C2 53.9 mm to (153.7, 70.6), turned to 180 degrees
- moved BZ1 52.1 mm to (160.1, 68.8), turned to 0 degrees
- moved C5 51.2 mm to (159.7, 84.4), turned to 0 degrees
- moved XL2 51.1 mm to (140.1, 72.5)
- moved C9 49.7 mm to (139.6, 57.2), turned to 0 degrees
- moved C7 47.8 mm to (161.4, 77.9)
- moved SW1 47.3 mm to (154.8, 60.0)
- moved C3 46.6 mm to (150.2, 70.6)
- moved C6 46.0 mm to (161.4, 81.8), turned to 90 degrees
- moved C10 43.0 mm to (142.7, 59.6), turned to -90 degrees
- moved DD1 42.5 mm to (153.2, 78.8), turned to 180 degrees
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Connections:
- net /LED_OUT renamed Net-(D4-PadC)
- BZ1 pad 1: PwrUnst -> +PwrUnst
- C1 pad 1: GND -> +PwrMCU
- C1 pad 2: +5V -> GND
- C10 pad 1: PwrMCU -> +PwrMCU
- C11 pad 1: PwrMCU -> GND
- C11 pad 2: GND -> /5V_MID
- C12 pad 1: PwrUnst -> GND
- C12 pad 2: GND -> +BATT
- C13 pad 1: PwrUnst -> Net-(C13-Pad1)
- C13 pad 2: GND -> Net-(C13-Pad2)
- C2 pad 1: GND -> +PwrMCU
- C2 pad 2: +5V -> GND
- C3 pad 1: PwrUnst -> +PwrMCU
- C4 pad 1: GND -> +PwrMCU
- C4 pad 2: +BATT -> GND
- C5 pad 1: PwrMCU -> +PwrMCU
- C6 pad 1: GND -> +PwrMCU
- C6 pad 2: PwrMCU -> GND
- C7 pad 1: PwrMCU -> Net-(C7-Pad1)
- C8 pad 1: PwrMCU -> Net-(C7-Pad1)
- C9 pad 1: PwrMCU -> +PwrUnst
- D1 pad A: +5V -> Net-(D1-PadA)
- D1 pad C: Net-(D1-PadC) -> GND
- D2 pad A: +5V -> /+5V_USB
- D2 pad C: /PWR_ALWAYS -> +PwrUnst
- D4 pad A: PwrUnst -> Net-(C13-Pad1)
- DA1 pad 1: /Charge -> GND
- DA1 pad 2: GND -> +PwrMCU
- DA1 pad 3: +BATT -> +PwrUnst
- DA2 pad 1: PwrUnst -> GND
- DA2 pad 2: GND -> Net-(DA2-Pad2)
- DA2 pad 3: PwrMCU -> GND
- DA2 pad 4: PwrUnst -> /5V_MID
- DD1 pad 1: PwrMCU -> +PwrMCU
- DD1 pad 10: Net-(DD1-Pad10) -> unconnected-(DD1-Pad10)
- DD1 pad 11: (no net) -> unconnected-(DD1-Pad11)
- DD1 pad 12: (no net) -> GND
- DD1 pad 13: (no net) -> Net-(C7-Pad1)
- DD1 pad 14: /LED_DAC -> Net-(DD1-Pad14)
- DD1 pad 15: (no net) -> /MeasEn
- DD1 pad 16: /LED_TIM -> /LED_V
- DD1 pad 17: (no net) -> /LED_CURR
- DD1 pad 18: (no net) -> GND
- DD1 pad 19: (no net) -> +PwrMCU
- DD1 pad 2: (no net) -> /USB_DETECT
- DD1 pad 20: (no net) -> /LED_CTRL
- DD1 pad 21: (no net) -> unconnected-(DD1-Pad21)
- DD1 pad 22: (no net) -> unconnected-(DD1-Pad22)
- DD1 pad 23: GND -> unconnected-(DD1-Pad23)
- DD1 pad 24: PwrMCU -> unconnected-(DD1-Pad24)
- DD1 pad 25: /DS1 -> /IS_CHARGING
- DD1 pad 26: /DS2 -> unconnected-(DD1-Pad26)
- DD1 pad 27: /DS3 -> unconnected-(DD1-Pad27)
- DD1 pad 28: /DS4 -> unconnected-(DD1-Pad28)
- DD1 pad 29: (no net) -> unconnected-(DD1-Pad29)
- DD1 pad 3: (no net) -> unconnected-(DD1-Pad3)
- DD1 pad 30: /UART_TX -> unconnected-(DD1-Pad30)
- DD1 pad 31: /UART_RX -> GND
- DD1 pad 32: /DS5 -> +PwrMCU
- DD1 pad 33: /DS6 -> unconnected-(DD1-Pad33)
- DD1 pad 34: /SWDIO -> unconnected-(DD1-Pad34)
- DD1 pad 35: GND -> Net-(DD1-Pad35)
- DD1 pad 36: PwrMCU -> unconnected-(DD1-Pad36)
- DD1 pad 37: /SWCLK -> /Buzzer
- DD1 pad 38: (no net) -> unconnected-(DD1-Pad38)
- DD1 pad 39: (no net) -> unconnected-(DD1-Pad39)
- DD1 pad 4: (no net) -> unconnected-(DD1-Pad4)
- DD1 pad 40: (no net) -> unconnected-(DD1-Pad40)
- DD1 pad 41: (no net) -> unconnected-(DD1-Pad41)
- DD1 pad 42: (no net) -> /UART_TX
- DD1 pad 43: (no net) -> /UART_RX
- DD1 pad 44: GND -> /USB_D-
- DD1 pad 45: (no net) -> /USB_D+
- DD1 pad 46: /Buzzer -> /SWDIO
- DD1 pad 48: PwrMCU -> +PwrMCU
- DD1 pad 5: (no net) -> unconnected-(DD1-Pad5)
- DD1 pad 6: (no net) -> unconnected-(DD1-Pad6)
- DD1 pad 7: (no net) -> unconnected-(DD1-Pad7)
- DD1 pad 8: GND -> unconnected-(DD1-Pad8)
- DD1 pad 9: PwrMCU -> unconnected-(DD1-Pad9)
- Q1 pad 1: +5V -> /+5V_USB
- Q1 pad 2: /PWR_ALWAYS -> +PwrUnst
- Q1 pad 3: +BATT -> Net-(Q1-Pad3)
- Q2 pad 1: Net-(Q2-Pad1) -> /Buzzer
- Q2 pad 2: /PWR_ALWAYS -> GND
- Q2 pad 3: PwrUnst -> /BuzzerOut
- Q4 pad 1: Net-(Q3-Pad2) -> /LED_CTRL
- Q4 pad 2: GND -> /LED_CURR
- Q5 pad 1: Net-(Q5-Pad1) -> /MeasEn
- Q5 pad 2: GND -> Net-(C13-Pad1)
- Q5 pad 3: /BuzzerOut -> Net-(Q5-Pad3)
- R1 pad 1: /Charge -> GND
- R1 pad 2: Net-(D1-PadC) -> Net-(R1-Pad2)
- R2 pad 1: Net-(DA1-Pad5) -> GND
- R2 pad 2: GND -> Net-(R2-Pad2)
- R3 pad 1: +5V -> Net-(D1-PadA)
- R3 pad 2: GND -> Net-(DD1-Pad35)
- R4 pad 1: Net-(F1-Pad1) -> /+5V_USB
- R4 pad 2: /LED_DAC -> /USB_DETECT
- R5 pad 1: Net-(Q3-Pad2) -> /USB_DETECT
- R6 pad 1: /Buzzer -> /+5V_USB
- R6 pad 2: Net-(Q5-Pad1) -> /5V_MID
- SW1 pad 1: Net-(DD1-Pad10) -> Net-(DD1-Pad14)
- SW1 pad 2: PwrMCU -> +PwrMCU
- SW1 pad H: (no net) -> GND
- XL1 pad 1: PwrMCU -> +PwrMCU
- XL2 pad 1: +5V -> GND
- XL2 pad 2: (no net) -> +BATT
Routing:
- net GND: track 332.0 -> 193.3 mm, vias 63 -> 84
- net +PwrMCU: track 0.00 -> 83.2 mm, vias 0 -> 5
- net /+5V_USB: track 0.00 -> 81.1 mm, vias 0 -> 2
- net PwrMCU: track 80.7 -> 0.00 mm, vias 4 -> 0
- net PwrUnst: track 51.6 -> 0.00 mm, vias 2 -> 0
- net /IS_CHARGING: track 0.00 -> 49.0 mm, vias 0 -> 2
- net +5V: track 46.8 -> 0.00 mm, vias 2 -> 0
- net Net-(DD1-Pad35): track 0.00 -> 45.3 mm, vias 0 -> 2
- net /USB_D+: track 0.00 -> 37.8 mm, vias 0 -> 3
- net /USB_D-: track 0.00 -> 37.1 mm, vias 0 -> 3
- net +PwrUnst: track 0.00 -> 35.8 mm, vias 0 -> 1
- net Net-(C13-Pad1): track 0.00 -> 29.3 mm
- net /USB_DETECT: track 0.00 -> 29.0 mm, vias 0 -> 2
- net /LED_V: track 0.00 -> 25.1 mm, vias 0 -> 2
- net Net-(DD1-Pad10): track 23.6 -> 0.00 mm, vias 1 -> 0
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Other:
- board size 30.2 x 53.5 mm -> 38 x 63 mm
- net class Default removed
- net class Wide removed
- rule pad_to_mask_clearance: 0.1 -> 0.06
- board text added: "-"
- board text added: "Avada5"

Commit message: PCB Layout Started
Parts:
- removed HOLE1, HOLE2, HOLE3, HOLE4: HOLE_METALLED, PCB:Hole2d2_out3d5mm
- removed Q4: DMG2302, SOT:SOT23-3A
- removed Q5: IRLML6401, SOT:SOT23-3
- removed R14, R16, R17, R18: 56k, Resistors:RES_0603
- removed R15: 0R1, Resistors:RES_1206
- removed R19: 2R0, Resistors:RES_0603
- added C16: 1u, Capacitors:CAP_0603_Silks, B.Cu at (199.3, 48.2)
- added D10: 2835, LEDs:LED_PLCC2835, F.Cu at (122.9, 76.5)
- added D11: 2835, LEDs:LED_PLCC2835, F.Cu at (126.9, 76.5)
- added D12: 2835, LEDs:LED_PLCC2835, F.Cu at (130.9, 76.5)
- added D13: 2835, LEDs:LED_PLCC2835, F.Cu at (134.9, 76.5)
- added D14: 2835, LEDs:LED_PLCC2835, F.Cu at (118.9, 81.5)
- added D15: 2835, LEDs:LED_PLCC2835, F.Cu at (122.9, 81.5)
- added D16: 2835, LEDs:LED_PLCC2835, F.Cu at (126.9, 81.5)
- added D17: 2835, LEDs:LED_PLCC2835, F.Cu at (130.9, 81.5)
- added D18: 2835, LEDs:LED_PLCC2835, F.Cu at (134.9, 81.5)
- added D19: 2835, LEDs:LED_PLCC2835, F.Cu at (122.9, 86.5)
- added D20: 2835, LEDs:LED_PLCC2835, F.Cu at (127.0, 86.5)
- added D21: 2835, LEDs:LED_PLCC2835, F.Cu at (130.9, 86.5)
- added D22: L-C191LBCT, LEDs:LED_0603, F.Cu at (118.3, 105.0)
- added D23: PMEG2020, Diodes:SOD323, B.Cu at (172.7, 53.2)
- added D3: 2835, LEDs:LED_PLCC2835, F.Cu at (130.9, 66.5)
- added D5: 2835, LEDs:LED_PLCC2835, F.Cu at (122.9, 71.5)
- added D6: 2835, LEDs:LED_PLCC2835, F.Cu at (126.9, 71.5)
- added D7: 2835, LEDs:LED_PLCC2835, F.Cu at (130.9, 71.5)
- added D8: 2835, LEDs:LED_PLCC2835, F.Cu at (134.9, 71.5)
- added D9: 2835, LEDs:LED_PLCC2835, F.Cu at (118.9, 76.5)
- added DA3: MCP1700, SOT:SOT23-3A, B.Cu at (164.7, 33.5)
- added Q3: IRLML6401, SOT:SOT23-3, B.Cu at (175.1, 65.0)
- added R10: 10k, Resistors:RES_0603, B.Cu at (195.2, 53.8)
- added R11: 56k, Resistors:RES_0603, B.Cu at (195.2, 56.5)
- added R13: 10k, Resistors:RES_0603, B.Cu at (195.2, 62.0)
- added R9: 0R2, Resistors:RES_1206, B.Cu at (169.9, 65.0)
- BZ1, C5, C6, DA2, DD1, L1, R3, R8, SA1, SW1, XL1: moved to B.Cu
- C1, C11: value 10u -> 1u; moved to B.Cu
- C10: value 1u -> 10n; moved to B.Cu
- C12: value 10u -> 2u2; moved to B.Cu
- C13, C14: value 3F -> 10u; footprint Capacitors:CAP_08xxR_HOR -> Capacitors:CAP_0603_Silks; moved to B.Cu
- C15: value 2u2 -> 1u; moved to B.Cu
- C2: value 0.1u -> 1u; moved to B.Cu
- C3: value 0.1u -> 3F; footprint Capacitors:CAP_0603_Silks -> Capacitors:CAP_08xxR_HOR; moved to B.Cu
- C4: value 0.1u -> 10u; moved to B.Cu
- C7: value 10n -> 0.1u; moved to B.Cu
- C8, C9: value 1u -> 0.1u; moved to B.Cu
- D1: value L-C191LBCT -> 2835; footprint LEDs:LED_0603 -> LEDs:LED_PLCC2835
- D2: value PMEG2020 -> 2835; footprint Diodes:SOD323 -> LEDs:LED_PLCC2835
- D4: value LEDwPAD -> 2835; footprint LEDs:LED_XPE -> LEDs:LED_PLCC2835
- DA1: value MCP1700 -> MCP1700-3002; moved to B.Cu
- Q1: value IRLML6401 -> IRLML0030; moved to B.Cu
- Q2: footprint SOT:SOT23-3A -> SOT:SOT23-3; moved to B.Cu
- R1: value 5k1 -> 20R; moved to B.Cu
- R12: value 20R -> 3k; moved to B.Cu
- R2: value 5k1 -> 56k; moved to B.Cu
- R4: value 10k -> 5k1; moved to B.Cu
- R5: value 10k -> 56k; moved to B.Cu
- R6: value 0R2 -> 2R0; footprint Resistors:RES_1206 -> Resistors:RES_0603; moved to B.Cu
- R7: value 3k -> 5k1; moved to B.Cu
- XL2: value CONN_2 -> 10PF-074; footprint Connectors:SLD_2_2D5 -> Connectors:USBC_10PF-074; moved to B.Cu
- XL3: value USB_C -> CONN_1; footprint Connectors:USB_C_MOLEX_1054500101 -> Connectors:PLS-1Square; moved to B.Cu
- XL4: value CONN_1 -> CONN_2; footprint Connectors:PLS-1Square -> Connectors:SLD_2_2D5; moved to B.Cu
- moved C12 92.6 mm to (203.5, 56.5), turned to 180 degrees
- moved R3 90.2 mm to (199.3, 56.5)
- moved R7 87.9 mm to (195.2, 48.2), turned to 180 degrees
- moved C11 87.3 mm to (203.5, 53.8), turned to 180 degrees
- moved XL3 86.2 mm to (175.4, 38.3), turned to 180 degrees
- moved XL4 82.3 mm to (167.8, 37.9), turned to 180 degrees
- moved R6 76.7 mm to (199.3, 64.8), turned to 180 degrees
- moved R1 76.1 mm to (199.3, 51.0), turned to 180 degrees
- moved R2 75.9 mm to (199.3, 53.8)
- moved C15 69.4 mm to (203.5, 64.8)
- moved C4 67.7 mm to (207.6, 53.8), turned to 180 degrees
- moved DA2 65.5 mm to (169.8, 59.2), turned to 180 degrees
- moved C9 64.5 mm to (203.5, 48.2), turned to 180 degrees
- moved C10 61.4 mm to (203.5, 51.0), turned to 180 degrees
- moved R4 59.7 mm to (199.3, 59.2), turned to 180 degrees
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Connections:
- C1 pad 1: +PwrMCU -> +BATT
- C10 pad 1: +PwrMCU -> Net-(DD1-VDDA)
- C11 pad 1: GND -> Net-(DD1-VDDA)
- C11 pad 2: /5V_MID -> GND
- C12 pad 1: GND -> Net-(C12-Pad1)
- C12 pad 2: +BATT -> GND
- C13 pad 1: Net-(C13-Pad1) -> GND
- C13 pad 2: Net-(C13-Pad2) -> /5V_MID
- C14 pad 1: Net-(C13-Pad2) -> GND
- C14 pad 2: GND -> +BATT
- C15 pad 1: Net-(C15-Pad1) -> +PwrUnst
- C2 pad 1: +PwrMCU -> Net-(DA1-OUT)
- C3 pad 1: +PwrMCU -> Net-(C3-Pad1)
- C7 pad 1: Net-(C7-Pad1) -> +PwrMCU
- C8 pad 1: Net-(C7-Pad1) -> +PwrMCU
- C9 pad 1: +PwrUnst -> +PwrMCU
- D1 pad A: Net-(D1-PadA) -> Net-(C3-Pad1)
- D1 pad C: GND -> Net-(Q1-D)
- D2 pad A: /+5V_USB -> Net-(C3-Pad1)
- D2 pad C: +PwrUnst -> Net-(Q1-D)
- D4 pad A: Net-(C13-Pad1) -> Net-(C3-Pad1)
- D4 pad C: Net-(D4-PadC) -> Net-(Q1-D)
- DA1 pad 2: +PwrMCU -> Net-(DA1-OUT)
- DA1 pad 3: +PwrUnst -> +BATT
- DA2 pad 2: Net-(DA2-Pad2) -> Net-(DA2-PROG)
- DD1 pad 13: Net-(C7-Pad1) -> Net-(DD1-VDDA)
- DD1 pad 15: /MeasEn -> /ADC_BAT
- DD1 pad 16: /LED_V -> unconnected-(DD1-ADC2/T15C1/T2C3/TX2/PA2-Pad16)
- DD1 pad 17: /LED_CURR -> unconnected-(DD1-ADC3/T15C2/T2C4/RX2/PA3-Pad17)
- DD1 pad 28: unconnected-(DD1-Pad28) -> /ADC_BAT_EN
- L1 pad 2: Net-(C7-Pad1) -> Net-(DD1-VDDA)
- Q1 pad 1: /+5V_USB -> /LED_CTRL
- Q1 pad 2: +PwrUnst -> GND
- Q1 pad 3: Net-(Q1-Pad3) -> Net-(Q1-D)
- R1 pad 1: GND -> Net-(DA1-OUT)
- R1 pad 2: Net-(R1-Pad2) -> Net-(C3-Pad1)
- R12 pad 1: +BATT -> Net-(DA2-PROG)
- R12 pad 2: Net-(C13-Pad1) -> GND
- R2 pad 1: GND -> /LED_CTRL
- R2 pad 2: Net-(R2-Pad2) -> GND
- R3 pad 1: Net-(D1-PadA) -> Net-(D22-PadA)
- R4 pad 1: /+5V_USB -> GND
- R4 pad 2: /USB_DETECT -> /USB_CC1_IN
- R5 pad 1: /USB_DETECT -> /Buzzer
- R6 pad 2: /5V_MID -> Net-(C12-Pad1)
- R7 pad 1: Net-(DA2-Pad2) -> /USB_CC2_IN
- R8 pad 1: /Buzzer -> +BATT
- R8 pad 2: GND -> /ADC_BAT
- SA1 pad 2: Net-(Q1-Pad3) -> Net-(Q3-D)
Routing:
- net GND: track 193.3 -> 0.00 mm, vias 84 -> 0
- net +PwrMCU: track 83.2 -> 0.00 mm, vias 5 -> 0
- net /+5V_USB: track 81.1 -> 0.00 mm, vias 2 -> 0
- net +BATT: track 51.9 -> 0.00 mm
- net /IS_CHARGING: track 49.0 -> 0.00 mm, vias 2 -> 0
- net Net-(DD1-PB14/MISO2/SDA2/T1C2N/T15C1): track 45.3 -> 0.00 mm, vias 2 -> 0
- net /USB_D+: track 37.8 -> 0.00 mm, vias 3 -> 0
- net /USB_D-: track 37.1 -> 0.00 mm, vias 3 -> 0
- net +PwrUnst: track 35.8 -> 0.00 mm, vias 1 -> 0
- net Net-(C13-Pad1): track 29.3 -> 0.00 mm
- net /USB_DETECT: track 29.0 -> 0.00 mm, vias 2 -> 0
- net /LED_V: track 25.1 -> 0.00 mm, vias 2 -> 0
- net /MeasEn: track 22.1 -> 0.00 mm, vias 2 -> 0
- net /LED_CURR: track 19.4 -> 0.00 mm, vias 2 -> 0
- net /SWCLK: track 18.1 -> 0.00 mm, vias 1 -> 0
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- removed copper zone on B.Cu, net GND
- removed copper zone on F.Cu, net GND
Other:
- outline, holes or cut-outs redrawn
- board text removed: "-"
- board text removed: "Avada5"

Commit message: + PCB sent to factory
Parts:
- removed C3: 3F, Capacitors:CAP_08xxR_HOR
- added XL5: CONN_1, Connectors:PLS-1Square, B.Cu at (122.0, 50.7)
- added XL6: CONN_1, Connectors:PLS-1Square, F.Cu at (140.1, 74.4)
- added XL7: CONN_1, Connectors:PLS-1Rnd, F.Cu at (143.6, 74.4)
- XL4: value CONN_2 -> CONN_1; footprint Connectors:SLD_2_2D5 -> Connectors:PLS-1Oval
- moved R3 96.0 mm to (116.5, 105.0), turned to 90 degrees
- moved R7 94.2 mm to (118.0, 102.2)
- moved XL3 91.6 mm to (109.2, 101.6)
- moved XL2 91.1 mm to (124.9, 102.8)
- moved C1 83.6 mm to (124.7, 58.7), turned to 90 degrees
- moved XL1 82.5 mm to (127.8, 47.0)
- moved C12 81.5 mm to (133.9, 98.9), turned to 0 degrees
- moved C7 80.8 mm to (126.8, 62.3)
- moved C2 80.5 mm to (127.3, 55.3)
- moved R4 79.9 mm to (130.9, 100.5)
- moved C14 78.5 mm to (131.4, 93.2)
- moved C6 78.4 mm to (131.0, 75.9), turned to 0 degrees
- moved R10 77.7 mm to (130.9, 97.3), turned to 0 degrees
- moved R6 76.5 mm to (130.9, 98.9), turned to 0 degrees
- moved C13 76.4 mm to (135.0, 93.2), turned to 0 degrees
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Connections:
- net Net-(C3-Pad1) renamed /+PwrLED
- net Net-(DA1-OUT) renamed /+3vLED
- net Net-(Q1-D) renamed /-PwrLED
- SA1 pad 1: unconnected-(SA1-Pad1) -> +BATT
- SA1 pad 3: +BATT -> unconnected-(SA1-Pad3)
- XL4 pad 1: GND -> +BATT
Routing:
- net GND: track 0.00 -> 233.5 mm, vias 0 -> 69
- net /+PwrLED: track 0.00 -> 120.5 mm, vias 0 -> 1
- net /-PwrLED: track 0.00 -> 102.8 mm, vias 0 -> 30
- net +PwrMCU: track 0.00 -> 94.7 mm, vias 0 -> 7
- net /+5V_USB: track 0.00 -> 76.2 mm, vias 0 -> 16
- net /USB_DETECT: track 0.00 -> 61.2 mm, vias 0 -> 2
- net +BATT: track 0.00 -> 57.3 mm, vias 0 -> 3
- net /USB_D+: track 0.00 -> 45.1 mm, vias 0 -> 2
- net /USB_D-: track 0.00 -> 43.8 mm, vias 0 -> 2
- net Net-(DD1-PB14/MISO2/SDA2/T1C2N/T15C1): track 0.00 -> 40.3 mm, vias 0 -> 2
- net /IS_CHARGING: track 0.00 -> 28.3 mm, vias 0 -> 2
- net +PwrUnst: track 0.00 -> 28.3 mm
- net /UART_RX: track 0.00 -> 25.6 mm, vias 0 -> 1
- net /UART_TX: track 0.00 -> 25.1 mm, vias 0 -> 1
- net /SWDIO: track 0.00 -> 22.5 mm, vias 0 -> 1
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- added copper zone on B.Cu, net +BATT
- added copper zone on F.Cu, net +BATT
- added copper zone on B.Cu, net /+5V_USB
- added copper zone on F.Cu, net /+5V_USB
- added copper zone on B.Cu, net /-PwrLED
- added copper zone on F.Cu, net /-PwrLED
- added copper zone on B.Cu, net GND
- added copper zone on F.Cu, net GND
Other:
- board text added: "+"
- board text added: "-"
